Commit message: fix RL using multi-agents

File: rotors_simulator/rotors_description/urdf/multirotor_base copy.xacro (robot description, xacro)
@@ -18,5 +18,4 @@
 <robot xmlns:xacro="http://ros.org/wiki/xacro">
   <!-- Macro for the inertia of a box -->
-    <xacro:property name="disable_collisions" value="true" />
   <xacro:macro name="box_inertia" params="x y z mass">
     <inertia ixx="${0.0833333 * mass * (y*y + z*z)}" ixy="0.0" ixz="0.0"
@@ -58,7 +57,10 @@
         </geometry>
       </visual>
-  <collision name="collision">
-    <geometry><box size="0.01 0.01 0.12"/></geometry> <!-- 缩小为极小体积 -->
-  </collision>
+    <collision>
+        <origin xyz="0 0 0" rpy="0 0 0" />
+        <geometry>
+          <box size="${body_width} ${body_width} ${body_height}" /> <!-- [m] [m] [m] -->
+        </geometry>
+      </collision>
     </link>
     <!-- attach multirotor_base_plugin to the base_link -->
@@ -101,7 +103,9 @@
         </geometry>
       </visual>
-  <collision name="collision">
-    <geometry><box size="0.01 0.01 0.12"/></geometry> <!-- 缩小为极小体积 -->
-  </collision>
+      <collision>
+        <geometry>
+          <cylinder length="0.005" radius="${radius_rotor}" /> <!-- [m] -->
+        </geometry>
+      </collision>
     </link>
     <gazebo>
