Commit message: perfect set no collision

File: rotors_simulator/rotors_description/urdf/component_snippets.xacro (robot description, xacro)
@@ -302,4 +302,7 @@
         <origin xyz="0 0 0" rpy="0 0 0" />
       </inertial>
+          <gazebo>
+    <disable_collisions>true</disable_collisions>
+  </gazebo>
     </link>
     <!-- IMU joint -->
@@ -345,4 +348,7 @@
         <mass value="${mass_odometry_sensor}" />  <!-- [kg] -->
       </inertial>
+          <gazebo>
+    <disable_collisions>true</disable_collisions>
+  </gazebo>
     </link>
     <!-- odometry joint -->
@@ -610,4 +616,7 @@
         <inertia ixx="1e-6" ixy="0" ixz="0" iyy="1e-6" iyz="0" izz="1e-6" />
       </inertial>
+       <gazebo>
+    <disable_collisions>true</disable_collisions>
+  </gazebo>
     </link>
     <joint name="${namespace}/camera_${camera_suffix}_joint" type="fixed">
@@ -674,4 +683,7 @@
         </geometry>
       </collision>
+ <gazebo>
+    <disable_collisions>true</disable_collisions>
+  </gazebo>
       <visual>
         <origin xyz="0 0 0" rpy="0 0 0" />

File: rotors_simulator/rotors_description/urdf/hummingbird.xacro (robot description, xacro)
@@ -17,4 +17,5 @@
 -->
 <robot name="hummingbird" xmlns:xacro="http://ros.org/wiki/xacro">
+  <xacro:property name="disable_collisions" value="true" />
   <!-- Properties (Taken from Novel Dynamic Inversion Architecture Design
 for Quadrocopter Control by Jian Wang et al.) -->

File: rotors_simulator/rotors_description/urdf/multirotor_base.xacro (robot description, xacro)
@@ -18,5 +18,6 @@
 <robot xmlns:xacro="http://ros.org/wiki/xacro">
   <!-- Macro for the inertia of a box -->
-    <xacro:property name="disable_collisions" value="true" />
+  <!-- 添加禁用碰撞属性 -->
+  <xacro:property name="disable_collisions" value="true" />
   <xacro:macro name="box_inertia" params="x y z mass">
     <inertia ixx="${0.0833333 * mass * (y*y + z*z)}" ixy="0.0" ixz="0.0"
@@ -58,7 +59,15 @@
         </geometry>
       </visual>
-  <collision name="collision">
-    <geometry><box size="0.01 0.01 0.12"/></geometry> <!-- 缩小为极小体积 -->
-  </collision>
+      <!-- 包裹碰撞节点 -->
+      <xacro:if value="${not disable_collisions}">
+        <collision name="collision">
+          <geometry>
+            <box size="0.01 0.01 0.12"/>
+          </geometry> <!-- 缩小为极小体积 -->
+        </collision>
+      </xacro:if>
+      <gazebo>
+        <disable_collisions>true</disable_collisions>
+      </gazebo>
     </link>
     <!-- attach multirotor_base_plugin to the base_link -->
@@ -91,17 +100,25 @@
           <!-- <cylinder length="0.005" radius="${radius_rotor}"/> --> <!-- [m] -->
           <xacro:if value="${use_own_mesh}">
-            <mesh filename="${mesh}"
-              scale="1 1 1" />
+            <mesh filename="${mesh}" scale="1 1 1" />
           </xacro:if>
           <xacro:unless value="${use_own_mesh}">
             <mesh filename="package://rotors_description/meshes/propeller_${direction}.dae"
-              scale="${radius_rotor} ${radius_rotor} ${radius_rotor}" /> <!-- The propeller meshes have a radius of 1m -->
+              scale="${radius_rotor} ${radius_rotor} ${radius_rotor}" />
+            <!-- The propeller meshes have a radius of 1m -->
             <!-- <box size="${2*radius_rotor} 0.01 0.005"/> -->
           </xacro:unless>
         </geometry>
       </visual>
-  <collision name="collision">
-    <geometry><box size="0.01 0.01 0.12"/></geometry> <!-- 缩小为极小体积 -->
-  </collision>
+      <!-- 包裹碰撞节点 -->
+      <xacro:if value="${not disable_collisions}">
+        <collision name="collision">
+          <geometry>
+            <box size="0.01 0.01 0.12"/>
+          </geometry> <!-- 缩小为极小体积 -->
+        </collision>
+      </xacro:if>
+      <gazebo>
+        <disable_collisions>true</disable_collisions>
+      </gazebo>
     </link>
     <gazebo>
@@ -127,4 +144,7 @@
       <material>Gazebo/${color}</material>
     </gazebo>
+    <gazebo>
+      <disable_collisions>true</disable_collisions>
+    </gazebo>
   </xacro:macro>
 </robot>
