Commit message: only position reward and step reward perform great

File: rotors_simulator/rotors_description/urdf/hummingbird.xacro (robot description, xacro)
@@ -17,5 +17,5 @@
 -->
 <robot name="hummingbird" xmlns:xacro="http://ros.org/wiki/xacro">
-  <xacro:property name="disable_collisions" value="true" />
+  <xacro:property name="disable_collisions" value="false" />
   <!-- Properties (Taken from Novel Dynamic Inversion Architecture Design
 for Quadrocopter Control by Jian Wang et al.) -->

Commit message: load stablebaselines3 PPO, change plot and model save

File: rotors_simulator/rotors_description/urdf/hummingbird.xacro (robot description, xacro)
@@ -17,5 +17,5 @@
 -->
 <robot name="hummingbird" xmlns:xacro="http://ros.org/wiki/xacro">
-  <xacro:property name="disable_collisions" value="false" />
+  <xacro:property name="disable_collisions" value="true" />
   <!-- Properties (Taken from Novel Dynamic Inversion Architecture Design
 for Quadrocopter Control by Jian Wang et al.) -->

File: rotors_simulator/rotors_description/urdf/multirotor_base.xacro (robot description, xacro)
@@ -19,5 +19,5 @@
   <!-- Macro for the inertia of a box -->
   <!-- 添加禁用碰撞属性 -->
-  <xacro:property name="disable_collisions" value="false" />
+  <xacro:property name="disable_collisions" value="true" />
   <xacro:macro name="box_inertia" params="x y z mass">
     <inertia ixx="${0.0833333 * mass * (y*y + z*z)}" ixy="0.0" ixz="0.0"
